File: electronics/prototype-test/prototype-test.kicad_pcb (KiCad board)
At the start: 2 copper layers, 0 parts

Commit message: finished prototype
Parts:
- added C1: 2u2, Capacitor_SMD:C_0603_1608Metric, F.Cu at (107.8, 98.4)
- added C10: 100n, Capacitor_SMD:C_0402_1005Metric, F.Cu at (111.1, 102.2)
- added C11: 2u2, Capacitor_SMD:C_0603_1608Metric, F.Cu at (109.3, 98.4)
- added C12: 100n, Capacitor_SMD:C_0402_1005Metric, F.Cu at (114.0, 114.9)
- added C13: 100n, Capacitor_SMD:C_0402_1005Metric, F.Cu at (111.2, 83.8)
- added C14: 30p, Capacitor_SMD:C_0402_1005Metric, F.Cu at (105.2, 112.1)
- added C15: 30p, Capacitor_SMD:C_0402_1005Metric, F.Cu at (99.8, 112.1)
- added C16: 10u, Capacitor_SMD:C_0805_2012Metric, F.Cu at (146.9, 88.0)
- added C17: 2u2, Capacitor_SMD:C_0603_1608Metric, F.Cu at (152.5, 97.3)
- added C18: 100n, Capacitor_SMD:C_0402_1005Metric, F.Cu at (151.2, 96.7)
- added C19: ?u, Capacitor_SMD:C_0805_2012Metric, F.Cu at (150.1, 89.3)
- added C2: 100n, Capacitor_SMD:C_0402_1005Metric, F.Cu at (105.5, 99.4)
- added C20: 100n, Capacitor_SMD:C_0402_1005Metric, F.Cu at (121.0, 89.5)
- added C21: 2u2, Capacitor_SMD:C_0603_1608Metric, F.Cu at (132.7, 85.7)
- added C3: 100n, Capacitor_SMD:C_0402_1005Metric, F.Cu at (107.1, 110.1)
- added C4: 100n, Capacitor_SMD:C_0402_1005Metric, F.Cu at (110.6, 99.4)
- added C5: 100n, Capacitor_SMD:C_0402_1005Metric, F.Cu at (106.6, 99.4)
- added C6: 100n, Capacitor_SMD:C_0402_1005Metric, F.Cu at (100.5, 102.2)
- added C7: 100n, Capacitor_SMD:C_0402_1005Metric, F.Cu at (100.5, 105.9)
- added C8: 100n, Capacitor_SMD:C_0402_1005Metric, F.Cu at (106.0, 110.1)
- added C9: 100n, Capacitor_SMD:C_0402_1005Metric, F.Cu at (112.3, 105.9)
- added D1: red, LED_SMD:LED_0603_1608Metric, F.Cu at (140.9, 59.6)
- added D2: green, LED_SMD:LED_0603_1608Metric, F.Cu at (142.5, 60.6)
- added D3: blue, LED_SMD:LED_0603_1608Metric, F.Cu at (144.2, 61.5)
- added D4: red, LED_SMD:LED_0603_1608Metric, F.Cu at (148.8, 125.1)
- added D5: green, LED_SMD:LED_0603_1608Metric, F.Cu at (150.3, 124.2)
- added D6: blue, LED_SMD:LED_0603_1608Metric, F.Cu at (151.8, 123.3)
- added D7: red, LED_SMD:LED_0603_1608Metric, F.Cu at (94.4, 89.4)
- added D8: green, LED_SMD:LED_0603_1608Metric, F.Cu at (94.4, 91.2)
- added D9: blue, LED_SMD:LED_0603_1608Metric, F.Cu at (94.4, 93.0)
- added J1: SolderPad, #TimGollLib:solder_pad_1.2x2.5mm, F.Cu at (126.4, 93.3)
- added J10: SolderPad, #TimGollLib:solder_pad_1.2x2.5mm, F.Cu at (130.2, 84.5)
- added J11: SolderPad, #TimGollLib:solder_pad_1.2x2.5mm, F.Cu at (130.2, 87.0)
- added J12: SolderPad, #TimGollLib:solder_pad_1.2x2.5mm, F.Cu at (126.4, 84.5)
- added J13: SolderPad, #TimGollLib:solder_pad_1.2x2.5mm, F.Cu at (126.4, 87.0)
- added J2: SolderPad, #TimGollLib:solder_pad_1.2x2.5mm, F.Cu at (126.4, 90.8)
- added J3: CortexDebug10, #TimGollLib:FTSH-105-01-F-DV-K, F.Cu at (118.7, 106.7)
- added J4: SolderPad, #TimGollLib:solder_pad_1.2x2.5mm, F.Cu at (126.4, 95.9)
- added J5: SolderPad, #TimGollLib:solder_pad_1.2x2.5mm, F.Cu at (126.4, 98.4)
- added J6: SolderPad, #TimGollLib:solder_pad_1.2x2.5mm, F.Cu at (130.2, 93.3)
- added J7: SolderPad, #TimGollLib:solder_pad_1.2x2.5mm, F.Cu at (130.2, 90.8)
- added J8: SolderPad, #TimGollLib:solder_pad_1.2x2.5mm, F.Cu at (130.2, 95.9)
- added J9: SolderPad, #TimGollLib:solder_pad_1.2x2.5mm, F.Cu at (130.2, 98.4)
- added MK1: Goertek B4013AM422-42, #TimGollLib:B4013AM422-42, F.Cu at (143.7, 84.8)
- added R1: 10k, Resistor_SMD:R_0603_1608Metric, F.Cu at (114.4, 116.2)
- added R10: 220, Resistor_SMD:R_0402_1005Metric, F.Cu at (96.9, 91.2)
- added R11: 120, Resistor_SMD:R_0402_1005Metric, F.Cu at (96.9, 93.0)
- added R12: 4k7, Resistor_SMD:R_0603_1608Metric, F.Cu at (121.3, 93.9)
- added R13: 4k7, Resistor_SMD:R_0603_1608Metric, F.Cu at (122.8, 93.9)
- added R2: 220, Resistor_SMD:R_0402_1005Metric, F.Cu at (139.6, 61.8)
- added R3: 220, Resistor_SMD:R_0402_1005Metric, F.Cu at (141.2, 62.8)
- added R4: 120, Resistor_SMD:R_0402_1005Metric, F.Cu at (142.9, 63.7)
- added R5: 220, Resistor_SMD:R_0402_1005Metric, F.Cu at (147.5, 122.9)
- added R6: 220, Resistor_SMD:R_0402_1005Metric, F.Cu at (149.0, 122.0)
- added R7: 2k2, Resistor_SMD:R_0805_2012Metric, F.Cu at (143.7, 89.3)
- added R8: 120, Resistor_SMD:R_0402_1005Metric, F.Cu at (150.6, 121.1)
- added R9: 220, Resistor_SMD:R_0402_1005Metric, F.Cu at (96.9, 89.4)
- added RV2: 100k, Potentiometer_THT:Potentiometer_Bourns_3296Y_Vertical, F.Cu at (149.4, 103.2)
- added SW1: reset, Button_Switch_SMD:SW_SPST_TL3342, F.Cu at (110.5, 120.0)
- added TP1: testpoint, #TimGollLib:tie-hook, F.Cu at (150.1, 84.2)
- added TP2: test, TestPoint:TestPoint_Pad_D1.5mm, F.Cu at (139.9, 103.3)
- added TP3: test, TestPoint:TestPoint_Pad_D1.5mm, F.Cu at (153.9, 103.3)
- added TP4: test, TestPoint:TestPoint_Pad_D1.5mm, F.Cu at (146.9, 109.6)
- added TP5: testpoint, #TimGollLib:tie-hook, F.Cu at (140.5, 96.3)
- added U1: W25Q128JVS, Package_SO:SOIC-8_5.275x5.275mm_P1.27mm, F.Cu at (106.0, 85.3)
- added U2: RP2040, Package_DFN_QFN:QFN-56-1EP_7x7mm_P0.4mm_EP3.2x3.2mm, F.Cu at (105.8, 104.8)
- added U4: LMC6482AIMX/NOPB, Package_SO:SOIC-8_3.9x4.9mm_P1.27mm, F.Cu at (146.9, 98.2)
- added U5: M24C02-WMN, Package_SO:SOIC-8_3.9x4.9mm_P1.27mm, F.Cu at (116.7, 90.9)
- added Y1: X322512MSB4SI, Crystal:Crystal_SMD_3225-4Pin_3.2x2.5mm, F.Cu at (102.5, 112.1)
Routing:
- net /LED_{blue,2}: track 0.00 -> 62.7 mm, vias 0 -> 2
- net /LED_{red,2}: track 0.00 -> 61.8 mm, vias 0 -> 2
- net /LED_{green,2}: track 0.00 -> 61.6 mm, vias 0 -> 2
- net /LED_{blue,1}: track 0.00 -> 60.3 mm, vias 0 -> 2
- net /mic_out: track 0.00 -> 59.4 mm, vias 0 -> 2
- net /LED_{green,1}: track 0.00 -> 57.1 mm, vias 0 -> 2
- net /LED_{red,1}: track 0.00 -> 56.4 mm, vias 0 -> 2
- net /mic_out_amp: track 0.00 -> 53.3 mm, vias 0 -> 2
- net /RPI_TX: track 0.00 -> 47.7 mm
- net +3V3: track 0.00 -> 44.2 mm, vias 0 -> 15
- net /RPI_RX: track 0.00 -> 44.0 mm
- net /RPI_TX_busy: track 0.00 -> 41.6 mm
- net /MCU/RUN: track 0.00 -> 30.1 mm, vias 0 -> 2
- net /SCL: track 0.00 -> 24.3 mm
- net /MCU/QSPI_SD3: track 0.00 -> 22.5 mm
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- added copper zone on B.Cu, net +3V3
- added copper zone on F.Cu, net GND
Other:
- board outline added: 103.9 x 119.1 mm
