File: electronics/prototype-test/prototype-test.kicad_sch (KiCad schematic)
At the start: 0 parts

Commit message: microphone circuit
Parts:
- added C16: 10u, Capacitor_SMD:C_0402_1005Metric, symbol Device:C_Small
- added C17: 2u2, Capacitor_SMD:C_0603_1608Metric, symbol Device:C_Small
- added C18: 100n, Capacitor_SMD:C_0402_1005Metric, symbol Device:C_Small
- added C19: ?u, Capacitor_SMD:C_0805_2012Metric, symbol Device:C_Small
- added MK1: Goertek B4013AM422-42, symbol Device:Microphone_Condenser
- added R7: 2k2, Resistor_SMD:R_0402_1005Metric, symbol Device:R_Small
- added RV2: 100k, Potentiometer_THT:Potentiometer_Bourns_3296Y_Vertical, symbol Device:R_Potentiometer_Small
- added TP1: testpoint, #TimGollLib:tie-hook, symbol Connector:TestPoint_Small
- added TP2, TP3, TP4: test, TestPoint:TestPoint_Pad_D1.5mm, symbol Connector:TestPoint_Small
- added U4: LMC6482AIMX/NOPB, Package_SO:SOIC-8_3.9x4.9mm_P1.27mm, symbol Amplifier_Operational:LMC6482
Connections:
- new net: C16.1, MK1.2 (+), R7.2
- new net: RV2.2, TP4.1, U4.2 (-)
- new net +3V3: R7.1
- new net +5VA: C17.1, C18.1, U4.8 (V+)
- new net GND: C17.2, C18.2, C19.2, MK1.1 (-), RV2.1, TP3.1, U4.4 (V-), U4.5 (+), U4.6 (-)
- new net mic_out: C16.2, C19.1, TP1.1, U4.3 (+)
- new net mic_out_amp: RV2.3, TP2.1, U4.1
- no-connect marks 0 -> 1
Other:
- added sheet MCU (hierarchical/mcu.kicad_sch)
- note added: "= mic_out * (1 + R1/R2)"
- note added: "maybe 0805 as well for prototyping"

Commit message: finished prototype
Parts:
- added C20: 100n, Capacitor_SMD:C_0402_1005Metric, symbol Device:C_Small
- added C21: 2u2, Capacitor_SMD:C_0603_1608Metric, symbol Device:C_Small
- added J1, J10, J11, J12, J13, J2, J4, J5, J6, J7, J8, J9: SolderPad, #TimGollLib:solder_pad_1.2x2.5mm, symbol Connector_Generic:Conn_01x01
- added R12, R13: 4k7, Resistor_SMD:R_0603_1608Metric, symbol Device:R_Small
- added TP5: testpoint, #TimGollLib:tie-hook, symbol Connector:TestPoint_Small
- added U5: M24C02-WMN, Package_SO:SOIC-8_3.9x4.9mm_P1.27mm, symbol Memory_EEPROM:M24C02-WMN
- C16: footprint Capacitor_SMD:C_0402_1005Metric -> Capacitor_SMD:C_0805_2012Metric; LCSC Part # C15525 -> C440198; Voltage 6.3V -> 50V
- MK1: footprint (none) -> #TimGollLib:B4013AM422-42
- R7: footprint Resistor_SMD:R_0402_1005Metric -> Resistor_SMD:R_0805_2012Metric; LCSC Part # C25879 -> C17520; Power 62.5mW -> 125mW
Connections:
- net +5VA is gone; now on net +3V3: C17.1, C18.1, U4.8 (V+)
- net +3V3: now also C20.1, C21.1, J10.1 (Pin_1), J12.1 (Pin_1), R12.1, R13.1, U5.8 (VCC)
- net GND: now also C20.2, C21.2, J11.1 (Pin_1), J13.1 (Pin_1), J5.1 (Pin_1), J9.1 (Pin_1), U5.1 (E0), U5.2 (E1), U5.3 (E2), U5.4 (VSS), U5.7 (~{WC})
- net mic_out_amp: now also TP5.1
- new net RPI_RX: J1.1 (Pin_1), J6.1 (Pin_1)
- new net RPI_TX: J2.1 (Pin_1), J7.1 (Pin_1)
- new net RPI_TX_busy: J4.1 (Pin_1), J8.1 (Pin_1)
- new net SCL: R13.2, U5.6 (SCL)
- new net SDA: R12.2, U5.5 (SDA)
Other:
- added sheet LEDs-1 (hierarchical/leds.kicad_sch)
- added sheet LEDs-2 (hierarchical/leds.kicad_sch)
- added sheet LEDs-3 (hierarchical/leds.kicad_sch)
- sheet MCU ports: added ADC_0, ADC_1, LED_{blue,1}, LED_{blue,2}, LED_{blue,3}, LED_{green,1}, LED_{green,2}, LED_{green,3}, LED_{red,1}, LED_{red,2}, LED_{red,3}, RX, SCL, SDA, TX, busy; removed none
- note added: "Amplifier"
- note added: "Connectors"
- note added: "EEPROM"
- note added: "LEDs"
- note added: "MCU"
- note added: "Microphone"
- note added: "address: 1010xyz, x:0, y:0, z:0 0x50"
- note added: "max current: LEDs: 3x3xm 5mA = 45mA MCU: ?mA MIC: negelectable"
- moved on the sheet: C16, C17, C18, C19, MK1, R7, RV2, TP1, TP2, TP3, TP4, U4A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
