File: electronics/prototype-test/hierarchical/mcu.kicad_sch (KiCad schematic)
At the start: 33 parts, among them J1 PinHeader, J2 PinHeader, J3 CortexDebug10, SW1 reset, U1 W25Q128JVS, U2 RP2040, U3 LM4040DBZ-3, Y1 X322512MSB4SI

Commit message: finished prototype
Parts:
- removed D1: SD03, Diode_SMD:D_SOD-323, symbol Device:D_Zener_Small
- removed D2: red, LED_SMD:LED_0603_1608Metric, symbol Device:LED_Small
- removed D3: blue, LED_SMD:LED_0603_1608Metric, symbol Device:LED_Small
- removed J1, J2: PinHeader, Connector_PinHeader_1.27mm:PinHeader_2x10_P1.27mm_Vertical_SMD, symbol Connector_Generic:Conn_02x10_Odd_Even
- removed JP1: LED_ENB, Jumper:SolderJumper-2_P1.3mm_Open_RoundedPad1.0x1.5mm, symbol Jumper:SolderJumper_2_Open
- removed R2, R3: 27R, Resistor_SMD:R_0603_1608Metric, symbol Device:R_Small
- removed R4: 10k, Resistor_SMD:R_0603_1608Metric, symbol Device:R_Small
- removed R5: 1k, Resistor_SMD:R_0603_1608Metric, symbol Device:R_Small
- removed R6: 220R, Resistor_SMD:R_0603_1608Metric, symbol Device:R_Small
- removed U3: LM4040DBZ-3, Package_TO_SOT_SMD:SOT-23, symbol Reference_Voltage:LM4040DBZ-3
- J3: footprint TimGollLib:FTSH-105-01-F-DV-K -> #TimGollLib:FTSH-105-01-F-DV-K; LCSC Part # C5250218 -> C3975188
Connections:
- net ADC_AVDD is gone; now on net +3V3: U2.43 (ADC_AVDD)
- net GPIO_00 renamed LED_{red,1}
- net GPIO_01 renamed LED_{red,2}
- net GPIO_02 renamed LED_{red,3}
- net GPIO_03 renamed LED_{green,1}
- net GPIO_04 renamed LED_{green,2}
- net GPIO_05 renamed LED_{green,3}
- net GPIO_06 renamed LED_{blue,1}
- net GPIO_07 renamed LED_{blue,2}
- net GPIO_08 renamed LED_{blue,3}
- net GPIO_16 renamed TX
- net GPIO_17 renamed RX
- net GPIO_18 renamed busy
- net GPIO_22 renamed SDA
- net GPIO_23 renamed SCL
- net GPIO_26 renamed ADC_0
- net GPIO_27 renamed ADC_1
- no-connect marks 1 -> 3
Other:
- note added: "used"
- note removed: "Analog Reference"
- note removed: "Pin Header"
- note removed: "Power & Status LEDs"
- note removed: "TODO!"
- note removed: "U_{LED,blue} = 3V1, I_{LED} = 1mA"
- note removed: "U_{LED,red} = 2V2, I_{LED} = 1mA"
- moved on the sheet: C1, C10, C11, C2, C3, C4, C5, C6, C7, C8, C9, J3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
