File: electronics/nerf-target-v1/nerf-target-v1.kicad_pcb (KiCad board)
At the start: 2 copper layers, 103.9 x 119.1 mm, 68 parts, among them J1 SolderPad, J10 SolderPad, J11 SolderPad, J12 SolderPad, J13 SolderPad, J2 SolderPad, J3 CortexDebug10, J4 SolderPad, J5 SolderPad, J6 SolderPad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

Commit message: finished board; production files
Parts:
- removed C12: 100n, Capacitor_SMD:C_0402_1005Metric
- removed R1: 10k, Resistor_SMD:R_0603_1608Metric
- removed SW1: reset, Button_Switch_SMD:SW_SPST_TL3342
- C14, C15: value 30p -> 33p
- moved R16 120.4 mm to (147.1, 96.5), turned to -90 degrees
- moved R18 118.8 mm to (149.4, 93.7)
- moved Q1 117.7 mm to (147.2, 100.2), turned to 90 degrees
- moved R17 117.2 mm to (146.3, 93.7)
- moved C17 116.1 mm to (148.8, 96.4), turned to -90 degrees
- moved TP2 114.1 mm to (142.9, 98.8)
- moved R14 112.0 mm to (145.8, 96.5), turned to -90 degrees
- moved R15 110.9 mm to (147.8, 91.8), turned to -90 degrees
- moved C21 8.76 mm to (124.0, 85.7)
Routing:
- net /MCU/GPIO_27: track 53.3 -> 0.00 mm, vias 2 -> 0
- net /mic_out: track 59.4 -> 8.74 mm, vias 2 -> 0
- net /mic_out_amp: track 0.00 -> 45.0 mm, vias 0 -> 2
- net Net-(Q1-B): track 0.00 -> 17.0 mm, vias 0 -> 2
- net (no net): track 16.7 -> 0.00 mm
- net /MCU/RUN: track 30.1 -> 17.5 mm
- net +3V3: track 44.2 -> 38.4 mm, vias 15 -> 14
- added copper zone on F.Cu, net Net-(Q1-B)
Other:
- board text added: "+3V3"
- board text added: "BUSY"
- board text added: "GND"
- board text added: "RX"
- board text added: "TX"
