File: electronics/nerf-target-v1/hierarchical/leds.kicad_sch (KiCad schematic)
At the start: 6 parts

Commit message: finished board; production files
Parts:
- D3: LCSC Part # C19171394 -> C965807
Changed lines of the file:
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@@
 			)
 		)
-		(property "LCSC Part #" "C19171394"
+		(property "LCSC Part #" "C965807"
 			(at 60.96 54.61 90)
 			(effects
